File: neftis/neftis.kicad_pcb (KiCad board)
At the start: 2 copper layers, 32 parts, among them Q1 BC847, Q2 BC847, U1 ESP32-S3-WROOM-1, U2 QRE1113, U3 QRE1113, U7 QRE1113, U8 QRE1113

Commit message: ponte H
Parts:
- removed 5v_to_3.3v1: AMS1117-3.3, Package_TO_SOT_SMD:SOT-223-3_TabPin2
- removed USB1: USB-B-S-X-X-TH, Library:USB-B
- removed serial1: Conn_01x02_Pin, Connector_PinHeader_2.54mm:PinHeader_1x02_P2.54mm_Vertical
- added AMS1117-3.3: 5v_to_3.3v, Package_TO_SOT_SMD:SOT-223-3_TabPin2, F.Cu at (143.7, 112.8)
- added Conn_01x02_Pin1: MOTOR_D, Connector_PinSocket_2.54mm:PinSocket_1x02_P2.54mm_Vertical, F.Cu at (166.8, 96.0)
- added Conn_01x02_Pin2: con_serial, Connector_PinHeader_2.54mm:PinHeader_1x02_P2.54mm_Vertical, F.Cu at (176.0, 96.0)
- added Conn_01x02_Pin3: MOTOR_D, Connector_PinSocket_2.54mm:PinSocket_1x02_P2.54mm_Vertical, F.Cu at (171.4, 96.0)
- added Conn_01x04_Pin1: ENC_D, Connector_PinSocket_2.54mm:PinSocket_1x04_P2.54mm_Vertical, F.Cu at (131.9, 110.9)
- added Conn_01x04_Pin2: ENC_D, Connector_PinSocket_2.54mm:PinSocket_1x04_P2.54mm_Vertical, F.Cu at (136.5, 110.9)
- added DRV8251ADDAR1: Ponte_H_E, Library:ponte_H, F.Cu at (168.7, 84.1)
- added DRV8251ADDAR2: Ponte_H_D, Library:ponte_H, F.Cu at (168.7, 90.5)
- added R10: 1.5k, Resistor_SMD:R_0805_2012Metric_Pad1.20x1.40mm_HandSolder, F.Cu at (157.4, 94.2)
- added R11: 1.5k, Resistor_SMD:R_0805_2012Metric_Pad1.20x1.40mm_HandSolder, F.Cu at (157.4, 97.1)
- added USB-B-S-X-X-TH1: USB_B, Library:USB-B, F.Cu at (158.7, 115.3)
- moved Q1 48.5 mm to (141.2, 119.3)
- moved Q2 48.5 mm to (141.2, 123.9)
- moved C1 38.1 mm to (145.7, 118.2)
- moved C5 38.1 mm to (145.7, 120.7)
- moved LM358 23.6 mm to (174.3, 104.8)
- moved U2 22.9 mm to (152.7, 105.1)
- moved U3 22.9 mm to (157.5, 105.1)
- moved U8 22.9 mm to (167.2, 105.1)
- moved U7 22.9 mm to (162.4, 105.1)
- moved R6 16.2 mm to (157.4, 82.3)
- moved R7 16.2 mm to (157.4, 85.3)
- moved R8 16.2 mm to (157.4, 88.2)
- moved R9 16.2 mm to (157.4, 91.2)
- moved RV1 15.5 mm to (171.5, 115.3)
- moved RV2 15.5 mm to (171.5, 123.5)
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Connections:
- U1 pad 20: unconnected-(U1-GPIO12/TOUCH12/ADC2_CH1/FSPICLK/FSPIIO6/SUBSPICLK-Pad20) -> D-
- U1 pad 21: unconnected-(U1-GPIO13/TOUCH13/ADC2_CH2/FSPIQ/FSPIIO7/SUBSPIQ-Pad21) -> D+
