File: projeto/projeto.kicad_pcb (KiCad board)
At the start: 2 copper layers, 40 parts, among them Q1 BC847, Q2 BC847, U1 ESP32-S3-WROOM-1, U2 QRE1113, U3 QRE1113, U7 QRE1113, U8 QRE1113

Commit message: quase ponto
Parts:
- removed AMS1117-3.3: 5v_to_3.3v, Package_TO_SOT_SMD:SOT-223-3_TabPin2
- removed DRV8251ADDAR1: Ponte_H_E, Library:ponte_H
- removed DRV8251ADDAR2: Ponte_H_D, Library:ponte_H
- removed LM358: Opamp_Dual, Library:LM358
- added BZ1: Buzzer, Buzzer_Beeper:Buzzer_12x9.5RM7.6, F.Cu at (149.4, 106.8)
- added C2: 100nF, Capacitor_SMD:C_0805_2012Metric_Pad1.18x1.45mm_HandSolder, F.Cu at (173.7, 86.8)
- added C3: 2.2µF, Capacitor_SMD:C_0805_2012Metric_Pad1.18x1.45mm_HandSolder, F.Cu at (173.7, 89.8)
- added C4: 10µF, Capacitor_SMD:C_0805_2012Metric_Pad1.18x1.45mm_HandSolder, F.Cu at (173.7, 92.8)
- added D4: LED, Resistor_SMD:R_0805_2012Metric_Pad1.20x1.40mm_HandSolder, F.Cu at (117.6, 99.6)
- added D5: LED, Resistor_SMD:R_0805_2012Metric_Pad1.20x1.40mm_HandSolder, F.Cu at (117.6, 102.5)
- added L1: 3.9µH, Inductor_SMD:L_APV_APH1040, F.Cu at (167.6, 105.8)
- added R12: 220, Resistor_SMD:R_0805_2012Metric_Pad1.20x1.40mm_HandSolder, F.Cu at (127.1, 96.6)
- added R15: 1.5k, Resistor_SMD:R_0805_2012Metric_Pad1.20x1.40mm_HandSolder, F.Cu at (127.1, 105.5)
- added R17: 220, Resistor_SMD:R_0805_2012Metric_Pad1.20x1.40mm_HandSolder, F.Cu at (127.1, 111.4)
- added R18: pull_up, Resistor_SMD:R_0805_2012Metric_Pad1.20x1.40mm_HandSolder, F.Cu at (131.8, 93.7)
- added R19: pull_up, Resistor_SMD:R_0805_2012Metric_Pad1.20x1.40mm_HandSolder, F.Cu at (131.8, 96.6)
- added R20: pull_up, Resistor_SMD:R_0805_2012Metric_Pad1.20x1.40mm_HandSolder, F.Cu at (131.8, 99.6)
- added R21: 220, Resistor_SMD:R_0805_2012Metric_Pad1.20x1.40mm_HandSolder, F.Cu at (131.8, 102.5)
- added R22: 100k, Resistor_SMD:R_1206_3216Metric, F.Cu at (172.0, 113.2)
- added R25: 33k, Resistor_SMD:R_1206_3216Metric, F.Cu at (172.0, 116.5)
- added SW1: btn2, Button_Switch_THT:SW_PUSH_6mm, F.Cu at (137.9, 84.3)
- added SW2: btn1, Button_Switch_THT:SW_PUSH_6mm, F.Cu at (137.9, 92.8)
- added SW3: btn3, Button_Switch_THT:SW_PUSH_6mm, F.Cu at (137.9, 101.4)
- added SW4: btn4, Button_Switch_THT:SW_PUSH_6mm, F.Cu at (137.9, 109.9)
- added SW6: SW_DPDT_x2, Button_Switch_THT:SW_CK_JS202011CQN_DPDT_Straight, F.Cu at (118.0, 122.2)
- added TP1: TP_12v, TestPoint:TestPoint_Pad_D1.5mm, F.Cu at (137.7, 66.3)
- added TP10: TP_IE, TestPoint:TestPoint_Pad_D1.5mm, F.Cu at (141.2, 80.5)
- added TP11: TP_ID, TestPoint:TestPoint_Pad_D1.5mm, F.Cu at (144.8, 66.3)
- added TP12: TP_IN1_E, TestPoint:TestPoint_Pad_D1.5mm, F.Cu at (144.8, 69.8)
- added TP13: TP_IN2_E, TestPoint:TestPoint_Pad_D1.5mm, F.Cu at (144.8, 73.4)
- added TP14: TP_IN2_D, TestPoint:TestPoint_Pad_D1.5mm, F.Cu at (144.8, 76.9)
- added TP15: TP_IN1_D, TestPoint:TestPoint_Pad_D1.5mm, F.Cu at (144.8, 80.5)
- added TP16: TP_DIV, TestPoint:TestPoint_Pad_D1.5mm, F.Cu at (148.3, 66.3)
- added TP17: TP_S0, TestPoint:TestPoint_Pad_D1.5mm, F.Cu at (148.3, 69.8)
- added TP18: TP_S1, TestPoint:TestPoint_Pad_D1.5mm, F.Cu at (148.3, 73.4)
- added TP19: TP_S2, TestPoint:TestPoint_Pad_D1.5mm, F.Cu at (148.3, 76.9)
- added TP2: TP_GND, TestPoint:TestPoint_Pad_D1.5mm, F.Cu at (137.7, 69.8)
- added TP20: TP_S3, TestPoint:TestPoint_Pad_D1.5mm, F.Cu at (148.3, 80.5)
- added TP21: TP_SIG, TestPoint:TestPoint_Pad_D1.5mm, F.Cu at (151.9, 66.3)
- added TP22: TP_BZR, TestPoint:TestPoint_Pad_D1.5mm, F.Cu at (151.9, 69.8)
- added TP23: TP_SE, TestPoint:TestPoint_Pad_D1.5mm, F.Cu at (151.9, 73.4)
- added TP24: TP_SD, TestPoint:TestPoint_Pad_D1.5mm, F.Cu at (151.9, 76.9)
- added TP25: TP_SED, TestPoint:TestPoint_Pad_D1.5mm, F.Cu at (151.9, 80.5)
- added TP26: TP_SDD, TestPoint:TestPoint_Pad_D1.5mm, F.Cu at (155.4, 66.3)
- added TP27: TP_SDA, TestPoint:TestPoint_Pad_D1.5mm, F.Cu at (155.4, 69.8)
- added TP28: TP_SEA, TestPoint:TestPoint_Pad_D1.5mm, F.Cu at (155.4, 73.4)
- added TP29: TP_REFD, TestPoint:TestPoint_Pad_D1.5mm, F.Cu at (155.4, 76.9)
- added TP3: TP_3V3, TestPoint:TestPoint_Pad_D1.5mm, F.Cu at (137.7, 73.4)
- added TP30: TP_REFE, TestPoint:TestPoint_Pad_D1.5mm, F.Cu at (155.4, 80.5)
- added TP4: TP_5V, TestPoint:TestPoint_Pad_D1.5mm, F.Cu at (137.7, 76.9)
- added TP5: TP_ME1, TestPoint:TestPoint_Pad_D1.5mm, F.Cu at (137.7, 80.5)
- added TP6: TP_ME2, TestPoint:TestPoint_Pad_D1.5mm, F.Cu at (141.2, 66.3)
- added TP7: TP_MD1, TestPoint:TestPoint_Pad_D1.5mm, F.Cu at (141.2, 69.8)
- added TP8: TP_MD2, TestPoint:TestPoint_Pad_D1.5mm, F.Cu at (141.2, 73.4)
- added TP9: TP_VM, TestPoint:TestPoint_Pad_D1.5mm, F.Cu at (141.2, 76.9)
- added U10: AP63203WU, Package_TO_SOT_SMD:TSOT-23-6, F.Cu at (165.9, 97.5)
- added U4: ICM-42688, Library:ICM-42688, F.Cu at (157.6, 115.6)
- added U5: DRV825, Library:DRV825, F.Cu at (167.3, 85.5)
- added U6: DRV825, Library:DRV825, F.Cu at (167.3, 91.9)
- added U9: LM358, Library:LM358, F.Cu at (140.6, 119.7)
- added con1: BATERIA, Connector_Samtec_HPM_THT:Samtec_HPM-02-01-x-S_Straight_1x02_Pitch5.08mm, F.Cu at (150.7, 117.1)
- added con7: MULTIPLEX, Connector_Molex:Molex_KK-254_AE-6410-07A_1x07_P2.54mm_Vertical, F.Cu at (117.5, 116.8)
- C1, C5: value 22 -> 22µF; footprint Capacitor_SMD:C_0603_1608Metric -> Capacitor_SMD:C_0805_2012Metric_Pad1.18x1.45mm_HandSolder
- Conn_01x02_Pin1: value MOTOR_D -> MOTOR_E
- R10: value 1.5k -> pull_up
- R3: value 100 -> 10k
- R9: value 10k -> 100
- RV1, RV2: footprint Potentiometer_THT:Potentiometer_Vishay_T73YP_Vertical_com3d -> Potentiometer_SMD:Potentiometer_Bourns_3314G_Vertical
- moved Q1 54.6 mm to (171.8, 74.1)
- moved Q2 54.6 mm to (171.8, 78.7)
- moved RV2 47.9 mm to (166.3, 75.9)
- moved Conn_01x02_Pin1 47.3 mm to (128.1, 123.0)
- moved Conn_01x02_Pin3 47.3 mm to (132.7, 123.0)
- moved C1 44.4 mm to (173.7, 83.8)
- moved R16 42.0 mm to (127.1, 108.4)
- moved RV1 41.0 mm to (160.2, 75.9)
- moved R14 40.5 mm to (127.1, 102.5)
- moved R6 39.1 mm to (122.3, 99.6)
- moved R7 39.1 mm to (122.3, 102.5)
- moved R1 39.1 mm to (117.6, 105.5)
- moved R10 39.1 mm to (122.3, 111.4)
- moved R2 39.1 mm to (117.6, 108.4)
- moved R3 39.1 mm to (117.6, 111.4)
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Connections:
- net Net-(LM358A-+) renamed SE_anal
- net Net-(LM358B-+) renamed SD_anal
- D1 pad 1: +5V -> Vin
- R10 pad 1: i_D -> +3.3V
- R10 pad 2: GND -> BTN_1
- R23 pad 1: RX -> TX
- R24 pad 2: TX -> RX
- R3 pad 2: Net-(U2-A) -> SE_digital
- R8 pad 2: Net-(U3-A) -> Net-(U2-A)
- R9 pad 2: SE_digital -> Net-(U3-A)
- U1 pad 27: unconnected-(U1-GPIO0/BOOT-Pad27) -> BOOT
- U1 pad 3: EN -> RST
- USB-B-S-X-X-TH1 pad 1: Net-(D1-A) -> +5V

Commit message: quase tudo SMD vida boa
Parts:
- removed SW4: btn4, Button_Switch_THT:SW_PUSH_6mm
- removed TP20: TP_S3, TestPoint:TestPoint_Pad_D1.5mm
- removed con7: MULTIPLEX, Connector_Molex:Molex_KK-254_AE-6410-07A_1x07_P2.54mm_Vertical
- added C10: 10µF, Capacitor_SMD:C_0805_2012Metric_Pad1.18x1.45mm_HandSolder, F.Cu at (181.0, 82.8)
- added C6: 0.1µF, Capacitor_SMD:C_0805_2012Metric_Pad1.18x1.45mm_HandSolder, F.Cu at (181.0, 70.8)
- added C7: 10nF, Capacitor_SMD:C_0805_2012Metric_Pad1.18x1.45mm_HandSolder, F.Cu at (181.0, 73.8)
- added C8: 0.1µF, Capacitor_SMD:C_0805_2012Metric_Pad1.18x1.45mm_HandSolder, F.Cu at (181.0, 76.8)
- added C9: 0.1µF, Capacitor_SMD:C_0805_2012Metric_Pad1.18x1.45mm_HandSolder, F.Cu at (181.0, 79.8)
- added D6: LED, Resistor_SMD:R_0805_2012Metric_Pad1.20x1.40mm_HandSolder, F.Cu at (123.3, 79.7)
- added J1: arrego, Connector_PinHeader_2.54mm:PinHeader_1x01_P2.54mm_Vertical, F.Cu at (180.9, 66.0)
- added J2: Conn_01x08_Pin, Connector_PinHeader_2.54mm:PinHeader_1x08_P2.54mm_Vertical, F.Cu at (176.4, 41.0)
- added P1: Card_SD, Library:Micro_SD_card, F.Cu at (163.3, 45.7)
- added R26: pull_up, Resistor_SMD:R_0805_2012Metric_Pad1.20x1.40mm_HandSolder, F.Cu at (137.5, 70.8)
- added R27: pull_up, Resistor_SMD:R_0805_2012Metric_Pad1.20x1.40mm_HandSolder, F.Cu at (137.5, 73.8)
- added R28: pull_up, Resistor_SMD:R_0805_2012Metric_Pad1.20x1.40mm_HandSolder, F.Cu at (137.5, 76.7)
- added R29: pull_up, Resistor_SMD:R_0805_2012Metric_Pad1.20x1.40mm_HandSolder, F.Cu at (137.5, 79.7)
- added R30: 220, Resistor_SMD:R_0805_2012Metric_Pad1.20x1.40mm_HandSolder, F.Cu at (137.5, 82.6)
- added SW5: SW_DPST_x2, Library:SW_SMD_6mm, F.Cu at (148.6, 65.5)
- added TP31: TP_ENC1_E, TestPoint:TestPoint_Pad_D1.0mm, F.Cu at (155.3, 73.8)
- added TP32: TP_ENC2_E, TestPoint:TestPoint_Pad_D1.0mm, F.Cu at (155.3, 76.9)
- added TP33: TP_ENC1_D, TestPoint:TestPoint_Pad_D1.0mm, F.Cu at (155.3, 80.0)
- added TP34: TP_ENC2_D, TestPoint:TestPoint_Pad_D1.0mm, F.Cu at (155.3, 83.0)
- added U11: CD4051B, Library:MUX, F.Cu at (169.0, 59.6)
- SW1: value btn2 -> SW_DPST_x2; footprint Button_Switch_THT:SW_PUSH_6mm -> Library:SW_SMD_6mm
- SW2: value btn1 -> SW_DPST_x2; footprint Button_Switch_THT:SW_PUSH_6mm -> Library:SW_SMD_6mm
- SW3: value btn3 -> SW_DPST_x2; footprint Button_Switch_THT:SW_PUSH_6mm -> Library:SW_SMD_6mm
- TP1, TP10, TP11, TP12, TP13, TP14, TP15, TP16, TP17, TP18, TP19, TP2, TP21, TP22, TP23, TP24, TP25, TP26, TP27, TP28, TP29, TP30, TP4, TP5, TP6, TP7, TP8, TP9: footprint TestPoint:TestPoint_Pad_D1.5mm -> TestPoint:TestPoint_Pad_D1.0mm
- TP3: value TP_3V3 -> TP_3.3V; footprint TestPoint:TestPoint_Pad_D1.5mm -> TestPoint:TestPoint_Pad_D1.0mm
- moved Conn_01x02_Pin1 70.7 mm to (157.3, 58.6)
- moved Conn_01x02_Pin3 70.7 mm to (161.9, 58.6)
- moved con1 69.9 mm to (182.9, 55.1)
- moved D1 66.4 mm to (168.2, 65.1)
- moved Conn_01x02_Pin2 57.3 mm to (176.4, 63.3)
- moved U5 46.2 mm to (182.6, 41.9)
- moved U6 46.2 mm to (182.6, 48.3)
- moved U7 46.1 mm to (133.0, 96.5)
- moved U2 46.1 mm to (123.4, 96.5)
- moved U3 46.1 mm to (128.2, 96.5)
- moved U8 46.1 mm to (137.8, 96.5)
- moved SW3 44.9 mm to (148.6, 57.8)
- moved SW2 44.0 mm to (148.6, 50.1)
- moved SW1 43.1 mm to (148.6, 42.5)
- moved R24 41.0 mm to (137.5, 67.9)
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Connections:
- R1 pad 1: +3V3 -> +3.3V
- R13 pad 1: +3V3 -> +3.3V
- R14 pad 2: +3V3 -> +3.3V
- R16 pad 1: +3V3 -> +3.3V
- R2 pad 2: +3V3 -> +3.3V
- R3 pad 1: +3V3 -> +3.3V
- R8 pad 1: +3V3 -> +3.3V
- R9 pad 1: +3V3 -> +3.3V
- RV1 pad 1: +3V3 -> +3.3V
- RV2 pad 1: +3V3 -> +3.3V
- SW2 pad 1: BTN_1 -> BTN_2
- SW3 pad 1: BTN_2 -> RST
- U1 pad 2: +3V3 -> +3.3V
- U9 pad 8: +3V3 -> +3.3V
Routing:
- net BTN_2: track 0.00 -> 2.35 mm
Other:
- board outline added: 94 x 85.5 mm
