File: projeto/projeto.kicad_sch (KiCad schematic)
At the start: 40 parts, among them Q1 BC847, Q2 BC847, U1 ESP32-S3-WROOM-1, U2 QRE1113, U3 QRE1113, U7 QRE1113, U8 QRE1113

Commit message: quase ponto
Parts:
- removed AMS1117-3.3: 5v_to_3.3v, Package_TO_SOT_SMD:SOT-223-3_TabPin2, symbol Regulator_Linear:AMS1117-3.3
- removed DRV8251ADDAR1: Ponte_H_E, Library:ponte_H, symbol DRV8251ADDAR:DRV8251ADDAR
- removed DRV8251ADDAR2: Ponte_H_D, Library:ponte_H, symbol DRV8251ADDAR:DRV8251ADDAR
- removed LM358: Opamp_Dual, Library:LM358, symbol Device:Opamp_Dual
- added BZ1: Buzzer, Buzzer_Beeper:Buzzer_12x9.5RM7.6, symbol Device:Buzzer
- added C2: 100nF, Capacitor_SMD:C_0805_2012Metric_Pad1.18x1.45mm_HandSolder, symbol Device:C
- added C3: 2.2µF, Capacitor_SMD:C_0805_2012Metric_Pad1.18x1.45mm_HandSolder, symbol Device:C
- added C4: 10µF, Capacitor_SMD:C_0805_2012Metric_Pad1.18x1.45mm_HandSolder, symbol Device:C
- added D4, D5: LED, Resistor_SMD:R_0805_2012Metric_Pad1.20x1.40mm_HandSolder, symbol Device:LED
- added L1: 3.9µH, Inductor_SMD:L_APV_APH1040, symbol Device:L
- added R12, R17, R21: 220, Resistor_SMD:R_0805_2012Metric_Pad1.20x1.40mm_HandSolder, symbol Device:R
- added R15: 1.5k, Resistor_SMD:R_0805_2012Metric_Pad1.20x1.40mm_HandSolder, symbol Device:R
- added R18, R19, R20: pull_up, Resistor_SMD:R_0805_2012Metric_Pad1.20x1.40mm_HandSolder, symbol Device:R
- added R22: 100k, Resistor_SMD:R_1206_3216Metric, symbol Device:R
- added R25: 33k, Resistor_SMD:R_1206_3216Metric, symbol Device:R
- added SW1: btn2, Button_Switch_THT:SW_PUSH_6mm, symbol Switch:SW_Push
- added SW2: btn1, Button_Switch_THT:SW_PUSH_6mm, symbol Switch:SW_Push
- added SW3: btn3, Button_Switch_THT:SW_PUSH_6mm, symbol Switch:SW_Push
- added SW4: btn4, Button_Switch_THT:SW_PUSH_6mm, symbol Switch:SW_Push
- added SW6: SW_DPDT_x2, Button_Switch_THT:SW_CK_JS202011CQN_DPDT_Straight, symbol Switch:SW_DPDT_x2
- added TP1: TP_12v, TestPoint:TestPoint_Pad_D1.5mm, symbol Connector:TestPoint
- added TP10: TP_IE, TestPoint:TestPoint_Pad_D1.5mm, symbol Connector:TestPoint
- added TP11: TP_ID, TestPoint:TestPoint_Pad_D1.5mm, symbol Connector:TestPoint
- added TP12: TP_IN1_E, TestPoint:TestPoint_Pad_D1.5mm, symbol Connector:TestPoint
- added TP13: TP_IN2_E, TestPoint:TestPoint_Pad_D1.5mm, symbol Connector:TestPoint
- added TP14: TP_IN2_D, TestPoint:TestPoint_Pad_D1.5mm, symbol Connector:TestPoint
- added TP15: TP_IN1_D, TestPoint:TestPoint_Pad_D1.5mm, symbol Connector:TestPoint
- added TP16: TP_DIV, TestPoint:TestPoint_Pad_D1.5mm, symbol Connector:TestPoint
- added TP17: TP_S0, TestPoint:TestPoint_Pad_D1.5mm, symbol Connector:TestPoint
- added TP18: TP_S1, TestPoint:TestPoint_Pad_D1.5mm, symbol Connector:TestPoint
- added TP19: TP_S2, TestPoint:TestPoint_Pad_D1.5mm, symbol Connector:TestPoint
- added TP2: TP_GND, TestPoint:TestPoint_Pad_D1.5mm, symbol Connector:TestPoint
- added TP20: TP_S3, TestPoint:TestPoint_Pad_D1.5mm, symbol Connector:TestPoint
- added TP21: TP_SIG, TestPoint:TestPoint_Pad_D1.5mm, symbol Connector:TestPoint
- added TP22: TP_BZR, TestPoint:TestPoint_Pad_D1.5mm, symbol Connector:TestPoint
- added TP23: TP_SE, TestPoint:TestPoint_Pad_D1.5mm, symbol Connector:TestPoint
- added TP24: TP_SD, TestPoint:TestPoint_Pad_D1.5mm, symbol Connector:TestPoint
- added TP25: TP_SED, TestPoint:TestPoint_Pad_D1.5mm, symbol Connector:TestPoint
- added TP26: TP_SDD, TestPoint:TestPoint_Pad_D1.5mm, symbol Connector:TestPoint
- added TP27: TP_SDA, TestPoint:TestPoint_Pad_D1.5mm, symbol Connector:TestPoint
- added TP28: TP_SEA, TestPoint:TestPoint_Pad_D1.5mm, symbol Connector:TestPoint
- added TP29: TP_REFD, TestPoint:TestPoint_Pad_D1.5mm, symbol Connector:TestPoint
- added TP3: TP_3V3, TestPoint:TestPoint_Pad_D1.5mm, symbol Connector:TestPoint
- added TP30: TP_REFE, TestPoint:TestPoint_Pad_D1.5mm, symbol Connector:TestPoint
- added TP31: TP_ENC1_E, TestPoint:TestPoint_Pad_D1.5mm, symbol Connector:TestPoint
- added TP32: TP_ENC2_E, TestPoint:TestPoint_Pad_D1.5mm, symbol Connector:TestPoint
- added TP33: TP_ENC1_D, TestPoint:TestPoint_Pad_D1.5mm, symbol Connector:TestPoint
- added TP34: TP_ENC2_D, TestPoint:TestPoint_Pad_D1.5mm, symbol Connector:TestPoint
- added TP4: TP_5V, TestPoint:TestPoint_Pad_D1.5mm, symbol Connector:TestPoint
- added TP5: TP_ME1, TestPoint:TestPoint_Pad_D1.5mm, symbol Connector:TestPoint
- added TP6: TP_ME2, TestPoint:TestPoint_Pad_D1.5mm, symbol Connector:TestPoint
- added TP7: TP_MD1, TestPoint:TestPoint_Pad_D1.5mm, symbol Connector:TestPoint
- added TP8: TP_MD2, TestPoint:TestPoint_Pad_D1.5mm, symbol Connector:TestPoint
- added TP9: TP_VM, TestPoint:TestPoint_Pad_D1.5mm, symbol Connector:TestPoint
- added U10: AP63203WU, Package_TO_SOT_SMD:TSOT-23-6, symbol Regulator_Switching:AP63203WU
- added U4: ICM-42688, Library:ICM-42688, symbol ICM-42688-P:ICM-42688-P
- added U5, U6: DRV825, Library:DRV825, symbol Driver_Motor:DRV8231ADSG
- added U9: LM358, Library:LM358, symbol Device:Opamp_Dual
- added con1: BATERIA, Connector_Samtec_HPM_THT:Samtec_HPM-02-01-x-S_Straight_1x02_Pitch5.08mm, symbol Connector:Conn_01x02_Socket
- added con7: MULTIPLEX, Connector_Molex:Molex_KK-254_AE-6410-07A_1x07_P2.54mm_Vertical, symbol Connector:Conn_01x07_Pin
- C1, C5: value 22 -> 22µF; footprint Capacitor_SMD:C_0603_1608Metric -> Capacitor_SMD:C_0805_2012Metric_Pad1.18x1.45mm_HandSolder
- Conn_01x02_Pin1: value MOTOR_D -> MOTOR_E
- R10: value 1.5k -> pull_up
- R3: value 100 -> 10k
- R9: value 10k -> 100
- RV1, RV2: footprint Potentiometer_THT:Potentiometer_Vishay_T73YP_Vertical_com3d -> Potentiometer_SMD:Potentiometer_Bourns_3314G_Vertical
Connections:
- net +12V: now also SW6.1 (A), SW6.4 (A), TP1.1, con1.1 (Pin_1)
- net +3.3V: now also R10.1, C3.1, L1.2, R18.1, R19.1, R20.1, TP3.1, U10.1 (FB), U4.12 (AP_CS), U4.5 (VDDIO), U4.8 (VDD), U5.4 (VREF), U6.4 (VREF)
- net +3V3: now also U9.8 (V+), con7.1 (Pin_1)
- net +5V: now also USB-B-S-X-X-TH1.1 (VCC), SW6.3 (C), SW6.6 (C), TP4.1; no longer D1.1 (K)
- net ENC1_D: now also TP33.1
- net ENC1_E: now also TP31.1
- net ENC2_D: now also TP34.1
- net ENC2_E: now also TP32.1
- net GND: now also BZ1.2 (+), C3.2, C4.1, R12.2, R15.2, R17.2, R25.1, SW1.2, SW2.2, SW3.2, SW4.2, TP2.1, U10.4 (GND), U4.1 (AP_SDO/AP_AD0), U4.11 (RESV_11), U4.6 (GND), U4.7 (RESV_7), U5.7 (GND), U5.9 (GND), U6.7 (GND), U6.9 (GND), U9.4 (V-), con1.2 (Pin_2), con7.7 (Pin_7); no longer R10.2
- net IN1_D: now also TP15.1, U6.3 (IN1)
- net IN1_E: now also TP12.1, U5.3 (IN1)
- net IN2_D: now also TP14.1, U6.2 (IN2)
- net IN2_E: now also TP13.1, U5.2 (IN2)
- net OUT1_D: now also TP8.1, U6.6 (OUT1)
- net OUT1_E: now also TP6.1, U5.6 (OUT1)
- net OUT2_D: now also TP7.1, U6.8 (OUT2)
- net OUT2_E: now also TP5.1, U5.8 (OUT2)
- net RX: now also R24.2, D5.2 (A); no longer R23.1
- net SD_digital: now also TP26.1
- net SE_digital: now also R3.2, TP25.1; no longer R9.2
- net TX: now also R23.1, D4.2 (A); no longer R24.2
- net i_D: now also R15.1, TP11.1, U6.1 (IPROPI); no longer R10.1
- net i_E: now also TP10.1, U5.1 (IPROPI)
- net BOOT: now reaches U1.27 (GPIO0/BOOT)
- net BOOT: now also R19.2, SW1.1
- net at RV1.2: now also TP29.1, U9.2 (-)
- net SD_anal: now reaches C5.2, R14.1, U7.3, U8.3
- net SD_anal: now also TP27.1, U9.3 (+)
- net at Q1.2 (B): now also TP24.1, U9.1
- net SE_anal: now reaches C1.2, R2.1, U2.3, U3.3
- net SE_anal: now also TP28.1, U9.5 (+)
- net at U2.1 (A): now also R8.2; no longer R3.2
- net at U3.1 (A): now also R9.2; no longer R8.2
- net at D1.2 (A): now also SW6.2 (B), SW6.5 (B); no longer USB-B-S-X-X-TH1.1 (VCC)
- net at Q2.2 (B): now also TP23.1, U9.7
- net at RV2.2: now also TP30.1, U9.6 (-)
- net EN renamed RST
- net RST: now also R20.2, SW4.1
- new net: D4.1 (K), R12.1
- new net: D5.1 (K), R17.1
- new net: C2.1, U10.6 (BST)
- new net: C2.2, L1.1, U10.5 (SW)
- new net: BZ1.1 (-), R21.1
- new net BTN_1: R10.2, SW2.1
- new net BTN_2: R18.2, SW3.1
- new net BZR: R21.2, TP22.1
- new net DIV_TENSAO: R22.1, R25.2, TP16.1
- new net S0: TP17.1, con7.3 (Pin_3)
- new net S1: TP18.1, con7.4 (Pin_4)
- new net S2: TP19.1, con7.5 (Pin_5)
- new net S3: TP20.1, con7.6 (Pin_6)
- new net SCL: U4.13 (AP_SCL/AP_SCLK)
- new net SDA: U4.14 (AP_SDA/AP_SDIO/AP_SDI)
- new net SIG: TP21.1, con7.2 (Pin_2)
- new net Vin: C4.2, D1.1 (K), R22.2, TP9.1, U10.2 (EN), U10.3 (IN), U5.5 (VM), U6.5 (VM)
- no-connect marks 2 -> 5

Commit message: quase tudo SMD vida boa
Parts:
- removed SW1: btn2, Button_Switch_THT:SW_PUSH_6mm, symbol Switch:SW_Push
- removed SW2: btn1, Button_Switch_THT:SW_PUSH_6mm, symbol Switch:SW_Push
- removed SW3: btn3, Button_Switch_THT:SW_PUSH_6mm, symbol Switch:SW_Push
- removed SW4: btn4, Button_Switch_THT:SW_PUSH_6mm, symbol Switch:SW_Push
- removed TP20: TP_S3, TestPoint:TestPoint_Pad_D1.5mm, symbol Connector:TestPoint
- removed con7: MULTIPLEX, Connector_Molex:Molex_KK-254_AE-6410-07A_1x07_P2.54mm_Vertical, symbol Connector:Conn_01x07_Pin
- added C10: 10µF, Capacitor_SMD:C_0805_2012Metric_Pad1.18x1.45mm_HandSolder, symbol Device:C
- added C6, C8, C9: 0.1µF, Capacitor_SMD:C_0805_2012Metric_Pad1.18x1.45mm_HandSolder, symbol Device:C
- added C7: 10nF, Capacitor_SMD:C_0805_2012Metric_Pad1.18x1.45mm_HandSolder, symbol Device:C
- added D6: LED, Resistor_SMD:R_0805_2012Metric_Pad1.20x1.40mm_HandSolder, symbol Device:LED
- added J1: arrego, Connector_PinHeader_2.54mm:PinHeader_1x01_P2.54mm_Vertical, symbol Connector:Conn_01x01_Pin
- added J2: Conn_01x08_Pin, Connector_PinHeader_2.54mm:PinHeader_1x08_P2.54mm_Vertical, symbol Connector:Conn_01x08_Pin
- added P1: Card_SD, Library:Micro_SD_card, symbol ST-TF-003A:ST-TF-003A
- added R26, R27, R28, R29: pull_up, Resistor_SMD:R_0805_2012Metric_Pad1.20x1.40mm_HandSolder, symbol Device:R
- added R30: 220, Resistor_SMD:R_0805_2012Metric_Pad1.20x1.40mm_HandSolder, symbol Device:R
- added SW1, SW2, SW3, SW5: SW_DPST_x2, Library:SW_SMD_6mm, symbol Switch:SW_DPST_x2
- added U11: CD4051B, Library:MUX, symbol Analog_Switch:CD4051B
- TP1, TP10, TP11, TP12, TP13, TP14, TP15, TP16, TP17, TP18, TP19, TP2, TP21, TP22, TP23, TP24, TP25, TP26, TP27, TP28, TP29, TP30, TP31, TP32, TP33, TP34, TP4, TP5, TP6, TP7, TP8, TP9: footprint TestPoint:TestPoint_Pad_D1.5mm -> TestPoint:TestPoint_Pad_D1.0mm
- TP3: value TP_3V3 -> TP_3.3V; footprint TestPoint:TestPoint_Pad_D1.5mm -> TestPoint:TestPoint_Pad_D1.0mm
Connections:
- net +3V3 is gone; now on net +3.3V: R1.1, R13.1, R14.2, R16.1, R2.2, R3.1, R8.1, R9.1, RV1.1, RV2.1, U1.2 (3V3), U9.8 (V+)
- net +3.3V: now also C10.1, C6.1, C7.1, C8.1, C9.1, D6.2 (A), J1.1 (Pin_1), P1.4 (VDD), R26.2, R27.2, R28.2, R29.2, U11.16 (VDD)
- net BOOT: now also SW1.1 (A), SW1.3 (A)
- net BTN_1: now also SW5.1 (A), SW5.3 (A)
- net BTN_2: now also SW2.1 (A), SW2.3 (A)
- net GND: now also C10.2, C6.2, C7.2, C8.2, C9.2, P1.6 (VSS), P1.G1 (GND), P1.G2 (GND), P1.G3 (GND), P1.G4 (GND), SW1.2 (B), SW1.4 (B), SW2.2 (B), SW2.4 (B), SW3.2 (B), SW3.4 (B), SW5.2 (B), SW5.4 (B), U11.6 (INH), U11.7 (VEE), U11.8 (VSS)
- net RST: now also SW3.1 (A), SW3.3 (A)
- net S0: now also U11.11 (A)
- net S1: now also U11.10 (B)
- net S2: now also U11.9 (C)
- net SIG: now also U11.3 (X)
- new net: D6.1 (K), R30.1
- new net: J2.4 (Pin_4), U11.1 (X4)
- new net: J2.5 (Pin_5), U11.12 (X3)
- new net: J2.8 (Pin_8), U11.13 (X0)
- new net: J2.7 (Pin_7), U11.14 (X1)
- new net: J2.6 (Pin_6), U11.15 (X2)
- new net: J2.2 (Pin_2), U11.2 (X6)
- new net: J2.1 (Pin_1), U11.4 (X7)
- new net: J2.3 (Pin_3), U11.5 (X5)
- new net CD: P1.9 (CD), R30.2
- new net CS: P1.2 (DAT3), R28.1
- new net MISO: P1.7 (DAT0), R26.1
- new net MOSI: P1.3 (CMD), R27.1
- new net SCK: P1.5 (CLK), R29.1
- no-connect marks 5 -> 7
